Commit message: [iCubGazeboV3] use simpified geom for foot collisions

File: iCub/robots/iCubGazeboV3/model.urdf (robot description, URDF)
Before this commit: robot iCub, 46 links, 45 joints
Links:
- link l_foot_front: geometry collision box size=0.1 0.117 0.010299988; visual mesh filename=package://iCub/meshes/simmechanics/sim_icub3_l_foot_front_p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 scale=0.001 0.001 0.001
- link l_foot_rear: geometry collision box size=0.1 0.117 0.010299988; visual mesh filename=package://iCub/meshes/simmechanics/sim_icub3_l_foot_rear_pr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 scale=0.001 0.001 0.001
- link r_foot_front: geometry collision box size=0.1 0.117 0.010299988; visual mesh filename=package://iCub/meshes/simmechanics/sim_icub3_r_foot_front_p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 scale=0.001 0.001 0.001
- link r_foot_rear: geometry collision box size=0.1 0.117 0.010299988; visual mesh filename=package://iCub/meshes/simmechanics/sim_icub3_r_foot_rear_pr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 scale=0.001 0.001 0.001
